Commit message: Husky Descript.

File: husky_ur_description/urdf/husky_ur5_e_description.urdf.xacro (robot description, xacro)
@@ -5,5 +5,5 @@
     <parent link="top_plate_front_link" />
     <child link="ur_arm_base_link" />
-    <origin xyz="$(optenv HUSKY_UR_XYZ -0.105 0.0 0.0)" rpy="$(optenv HUSKY_UR_RPY 0 0 3.1415927)"/>
+    <origin xyz="$(optenv HUSKY_UR_XYZ -0.105 0.0 0.0)" rpy="$(optenv HUSKY_UR_RPY 0 0 -1.5708)"/>
   </joint>
   <xacro:ur5e_robot prefix="ur_arm_" joint_limited="true"/>
